File: Hardware/RGB Panel Shield for Arduino.sch (EAGLE design)
At the start: 13 parts, among them J7 Screw Terminal, J8 SparkFun Panel, U1 ARDUINO UNO

Commit message: Readme fix
Parts:
- added U$91: SPARKX-LOGO4, SparkX:SPARKX-LOGO4
Other:
- moved on the sheet: J2, J3, J4, J6, J7, J8, U1
